Commit message: fix pure pursuit

File: catkin_ws/src/models/bot/urdf/bot.xacro (robot description, xacro)
@@ -323,3 +323,7 @@
     <child link="camera"/>
   </joint>
+  <xacro:include filename="$(find velodyne_description)/urdf/VLP-16.urdf.xacro"/>
+  <VLP-16 parent="base_link" name="velodyne" topic="/velodyne_points" hz="10" samples="440">
+    <origin xyz="0 0 0.05" rpy="0 0 0" />
+  </VLP-16>
 </robot>
