Commit message: test gazebo car model(failed)

File: catkin_ws/src/robot/bot/urdf/bot.xacro (robot description, xacro)
@@ -121,19 +121,19 @@
       <geometry>
         <mesh
-          filename="package://duckiebot_1/meshes/base_link.STL" />
-      </geometry>
-      <material
-        name="">
-        <color
-          rgba="0.792156862745098 0.819607843137255 0.933333333333333 1" />
-      </material>
-    </visual>
-    <collision>
-      <origin
-        xyz="0 0 0"
-        rpy="0 0 0" />
-      <geometry>
-        <mesh
-          filename="package://duckiebot_1/meshes/base_link.STL" />
+          filename="package://bot/meshes/base_link.STL" />
+      </geometry>
+      <material
+        name="">
+        <color
+          rgba="0.792156862745098 0.819607843137255 0.933333333333333 1" />
+      </material>
+    </visual>
+    <collision>
+      <origin
+        xyz="0 0 0"
+        rpy="0 0 0" />
+      <geometry>
+        <mesh
+          filename="package://bot/meshes/base_link.STL" />
       </geometry>
     </collision>
@@ -161,19 +161,19 @@
       <geometry>
         <mesh
-          filename="package://duckiebot_1/meshes/lwheel_link.STL" />
-      </geometry>
-      <material
-        name="">
-        <color
-          rgba="0.792156862745098 0.819607843137255 0.933333333333333 1" />
-      </material>
-    </visual>
-    <collision>
-      <origin
-        xyz="0 0 0"
-        rpy="0 0 0" />
-      <geometry>
-        <mesh
-          filename="package://duckiebot_1/meshes/lwheel_link.STL" />
+          filename="package://bot/meshes/lwheel_link.STL" />
+      </geometry>
+      <material
+        name="">
+        <color
+          rgba="0.792156862745098 0.819607843137255 0.933333333333333 1" />
+      </material>
+    </visual>
+    <collision>
+      <origin
+        xyz="0 0 0"
+        rpy="0 0 0" />
+      <geometry>
+        <mesh
+          filename="package://bot/meshes/lwheel_link.STL" />
       </geometry>
     </collision>
@@ -214,19 +214,19 @@
       <geometry>
         <mesh
-          filename="package://duckiebot_1/meshes/rwheel_link.STL" />
-      </geometry>
-      <material
-        name="">
-        <color
-          rgba="0.792156862745098 0.819607843137255 0.933333333333333 1" />
-      </material>
-    </visual>
-    <collision>
-      <origin
-        xyz="0 0 0"
-        rpy="0 0 0" />
-      <geometry>
-        <mesh
-          filename="package://duckiebot_1/meshes/rwheel_link.STL" />
+          filename="package://bot/meshes/rwheel_link.STL" />
+      </geometry>
+      <material
+        name="">
+        <color
+          rgba="0.792156862745098 0.819607843137255 0.933333333333333 1" />
+      </material>
+    </visual>
+    <collision>
+      <origin
+        xyz="0 0 0"
+        rpy="0 0 0" />
+      <geometry>
+        <mesh
+          filename="package://bot/meshes/rwheel_link.STL" />
       </geometry>
     </collision>
@@ -267,19 +267,19 @@
       <geometry>
         <mesh
-          filename="package://duckiebot_1/meshes/wheelconnect_link.STL" />
-      </geometry>
-      <material
-        name="">
-        <color
-          rgba="0.792156862745098 0.819607843137255 0.933333333333333 1" />
-      </material>
-    </visual>
-    <collision>
-      <origin
-        xyz="0 0 0"
-        rpy="0 0 0" />
-      <geometry>
-        <mesh
-          filename="package://duckiebot_1/meshes/wheelconnect_link.STL" />
+          filename="package://bot/meshes/wheelconnect_link.STL" />
+      </geometry>
+      <material
+        name="">
+        <color
+          rgba="0.792156862745098 0.819607843137255 0.933333333333333 1" />
+      </material>
+    </visual>
+    <collision>
+      <origin
+        xyz="0 0 0"
+        rpy="0 0 0" />
+      <geometry>
+        <mesh
+          filename="package://bot/meshes/wheelconnect_link.STL" />
       </geometry>
     </collision>
@@ -320,19 +320,19 @@
       <geometry>
         <mesh
-          filename="package://duckiebot_1/meshes/swheel_link.STL" />
-      </geometry>
-      <material
-        name="">
-        <color
-          rgba="0.792156862745098 0.819607843137255 0.933333333333333 1" />
-      </material>
-    </visual>
-    <collision>
-      <origin
-        xyz="0 0 0"
-        rpy="0 0 0" />
-      <geometry>
-        <mesh
-          filename="package://duckiebot_1/meshes/swheel_link.STL" />
+          filename="package://bot/meshes/swheel_link.STL" />
+      </geometry>
+      <material
+        name="">
+        <color
+          rgba="0.792156862745098 0.819607843137255 0.933333333333333 1" />
+      </material>
+    </visual>
+    <collision>
+      <origin
+        xyz="0 0 0"
+        rpy="0 0 0" />
+      <geometry>
+        <mesh
+          filename="package://bot/meshes/swheel_link.STL" />
       </geometry>
     </collision>

File: catkin_ws/src/robot/duckiecar/urdf/duckiecar.xacro (robot description, xacro)
@@ -105,7 +105,7 @@
       <origin
         xyz="-0.0153668055531249 4.44089209850063E-16 -0.0534671165486267"
-        rpy="0 -3.14 0" />
-      <mass
-        value="22.4144467859455" /> <!--947.122649398591-->
+        rpy="0 0 0" />
+      <mass
+        value="9.47122649398591" />
       <inertia
         ixx="301.370472338624"
@@ -147,5 +147,5 @@
         rpy="0 0 0" />
       <mass
-        value="5.57789775644867" /> <!--56.5329598013484-->
+        value="5.65329598013484" />
       <inertia
         ixx="1.46078812586693"
@@ -191,5 +191,5 @@
       link="lwheel_link" />
     <axis
-      xyz="0 -1 0" />
+      xyz="0 1 0" />
   </joint>
   <link
@@ -200,5 +200,5 @@
         rpy="0 0 0" />
       <mass
-        value="5.57789775644867" />
+        value="5.65329598013484" />
       <inertia
         ixx="1.46078812586693"
@@ -244,5 +244,5 @@
       link="rwheel_link" />
     <axis
-      xyz="0 -1 0" />
+      xyz="0 1 0" />
   </joint>
   <link
@@ -253,5 +253,5 @@
         rpy="0 0 0" />
       <mass
-        value="12.2264377536546" />
+        value="0.122264377536546" />
       <inertia
         ixx="0.353513318523549"
@@ -306,5 +306,5 @@
         rpy="0 0 0" />
       <mass
-        value="11.8409774219159" />
+        value="0.118409774219159" />
       <inertia
         ixx="0.090404402128395"
@@ -350,35 +350,5 @@
       link="swheel_link" />
     <axis
-      xyz="0 -1 0" />
+      xyz="0 1 0" />
   </joint>
-  <link name="camera">
-    <collision>
-      <origin rpy="0 0.1 0" xyz="0 0 0"/>
-      <geometry>
-        <box size="0.02 0.02 0.02"/>
-      </geometry>
-    </collision>
-    <visual>
-      <origin rpy="0 0 0" xyz="0 0 0"/>
-      <geometry>
-        <box size="0.02 0.02 0.02"/>
-      </geometry>
-    </visual>
-    <inertial>
-      <mass value="0.01"/>
-      <origin rpy="0 0 0" xyz="0 0 0"/>
-      <box_inertia m="0.1" x="0.02" y="0.02" z="0.02"/>
-      <inertia ixx="1e-6" ixy="0" ixz="0" iyy="1e-6" iyz="0" izz="1e-6"/>
-    </inertial>
-  </link>
-  <joint name="camera_joint" type="fixed">
-    <axis xyz="0 0 0"/>
-    <origin rpy="0 0.9 0" xyz=".12 0 .1"/>
-    <parent link="base_link"/>
-    <child link="camera"/>
-  </joint>
-  <xacro:include filename="$(find velodyne_description)/urdf/VLP-16.urdf.xacro"/>
-  <VLP-16 parent="base_link" name="velodyne" topic="/velodyne_points" hz="10" samples="440">
-    <origin xyz="1.5 0 0.05" rpy="0 0 0" />
-  </VLP-16>
 </robot>
